File: circuit/main/main.kicad_sch (KiCad schematic)
At the start: 21 parts, among them J1 XT30, J2 GP1UXC41QS, J3 Barrel_Jack_MountingPin, M1 Motor_Servo_JR, M2 Motor_Servo_JR, M3 Motor_Servo_JR, M4 Motor_Servo_JR, M5 Motor_Servo_JR, SW1 SW_Push

Commit message: 回路
Parts:
- removed J3: Barrel_Jack_MountingPin, symbol Connector:Barrel_Jack_MountingPin
- added Q1: IRF9383M, Package_DirectFET:DirectFET_MX, symbol Transistor_FET:IRF9383M
- added R5: R_Small, symbol Device:R_Small
Connections:
- net +BATT: now also Q1.1 (D); no longer J1.1 (Pin_1)
- net GND: now also Q1.2 (G), R5.2
- new net: J1.1 (Pin_1), Q1.3 (S), R5.1
- no-connect marks 3 -> 2
Other:
- moved on the sheet: A1, C1, C2, C3, D1, D2, D3, J2, M1, M2, M3, M4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

Commit message: フットプリント割当
Parts:
- removed Q1: IRF9383M, Package_DirectFET:DirectFET_MX, symbol Transistor_FET:IRF9383M
- added C4: 47u, Capacitor_THT:CP_Radial_D5.0mm_P2.00mm, symbol Device:C_Polarized_Small
- added J3: NeoPixel, Connector_JST:JST_PH_B3B-PH-K_1x03_P2.00mm_Vertical, symbol Connector_Generic:Conn_01x03
- added SW3: SW_SPDT, Button_Switch_THT:SW_Slide_SPDT_Angled_CK_OS102011MA1Q, symbol Switch:SW_SPDT
- added U2: ~, Package_SO:TSOP-6_1.65x3.05mm_P0.95mm, symbol Transistor_FET:SSM6J808R
- C1: footprint (none) -> Capacitor_SMD:C_0603_1608Metric_Pad1.08x0.95mm_HandSolder
- C2, C3: footprint (none) -> Capacitor_THT:CP_Radial_D5.0mm_P2.00mm
- D1, D2, D3: footprint (none) -> LED_SMD:LED_0603_1608Metric_Pad1.05x0.95mm_HandSolder
- J1: footprint (none) -> Connector_AMASS:AMASS_XT30PW-M_1x02_P2.50mm_Horizontal
- J2: footprint (none) -> Button_Switch_THT:SW_MEC_5GTH9
- M1, M2, M3, M4, M5: footprint (none) -> Connector_PinSocket_2.54mm:PinSocket_1x03_P2.54mm_Vertical
- R1, R2, R3, R4, R5: footprint (none) -> Resistor_SMD:R_0603_1608Metric_Pad0.98x0.95mm_HandSolder
- SW1: footprint (none) -> Button_Switch_THT:SW_PUSH-12mm
Connections:
- net +BATT: now also C4.1, J3.1 (Pin_1), U2.1 (D), U2.2 (D), U2.5 (D), U2.6 (D)
- net GND: now also C4.2, J3.3 (Pin_3), SW3.3 (C); no longer R5.2
- net IR_SIGNAL: now also J2.1 (Pin_1); no longer J2.3 (Pin_3)
- net at R1.2: now also J2.3 (Pin_3); no longer J2.1 (Pin_1)
- net at J1.1 (Pin_1), R5.1: now also U2.4 (S)
- net NEOPIXEL_SIGNAL: now reaches A1.9 (D6)
- net NEOPIXEL_SIGNAL: now also J3.2 (Pin_2)
- new net: R5.2, SW3.2 (B), U2.3 (G)
- no-connect marks 2 -> 19
Other:
- moved on the sheet: C2, J2, R1

Commit message: パターン図
Parts:
- J2: footprint Button_Switch_THT:SW_MEC_5GTH9 -> OptoDevice:Vishay_MINICAST-3Pin
- M1, M2, M3, M4, M5: footprint Connector_PinSocket_2.54mm:PinSocket_1x03_P2.54mm_Vertical -> Connector_PinHeader_2.54mm:PinHeader_1x03_P2.54mm_Vertical
Connections:
- net +5V: now also C4.1
- net +BATT: no longer C4.1
- net GND: now also J1.1 (Pin_1); no longer J1.2 (Pin_2)
- net PWM0: now also A1.14 (D11); no longer A1.6 (D3)
- net PWM1: now also A1.13 (D10); no longer A1.8 (D5)
- net PWM3: now also A1.8 (D5); no longer A1.13 (D10)
- net PWM4: now also A1.6 (D3); no longer A1.14 (D11)
- net at R5.1, U2.4 (S): now also J1.2 (Pin_2); no longer J1.1 (Pin_1)
Other:
- moved on the sheet: J1
Changed lines of the file:
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@@
 	)
 	(junction
-		(at 240.03 76.2)
-		(diameter 0)
-		(color 0 0 0 0)
-	)
-	(junction
 		(at 173.99 116.84)
 		(diameter 0)
@@
 	)
 	(junction
-		(at 240.03 68.58)
+		(at 243.84 36.83)
 		(diameter 0)
 		(color 0 0 0 0)
 	)
 	(junction
-		(at 243.84 36.83)
+		(at 173.99 88.9)
 		(diameter 0)
 		(color 0 0 0 0)
 	)
 	(junction
-		(at 173.99 88.9)
+		(at 184.15 153.67)
 		(diameter 0)
 		(color 0 0 0 0)
@@
 	)
 	(junction
+		(at 173.99 144.78)
+		(diameter 0)
+		(color 0 0 0 0)
+	)
+	(junction
 		(at 243.84 29.21)
 		(diameter 0)
@@
 	(wire
 		(pts
-			(xy 240.03 74.93) (xy 240.03 76.2)
-		)
-		(stroke
-			(width 0)
-			(type default)
-		)
-	)
-	(wire
-		(pts
 			(xy 92.71 97.79) (xy 92.71 99.06)
 		)
@@
 	(wire
 		(pts
+			(xy 173.99 144.78) (xy 173.99 147.32)
+		)
+		(stroke
+			(width 0)
+			(type default)
+		)
+	)
+	(wire
+		(pts
 			(xy 243.84 25.4) (xy 243.84 29.21)
 		)
@@
 	(wire
 		(pts
+			(xy 173.99 152.4) (xy 173.99 153.67)
+		)
+		(stroke
+			(width 0)
+			(type default)
+		)
+	)
+	(wire
+		(pts
 			(xy 184.15 105.41) (xy 191.77 105.41)
 		)
@@
 	(wire
 		(pts
-			(xy 184.15 154.94) (xy 184.15 147.32)
+			(xy 184.15 154.94) (xy 184.15 153.67)
 		)
 		(stroke
@@
 	(wire
 		(pts
-			(xy 240.03 68.58) (xy 240.03 69.85)
+			(xy 127 105.41) (xy 127 109.22)
 		)
 		(stroke
@@
 	(wire
 		(pts
-			(xy 127 105.41) (xy 127 109.22)
+			(xy 57.15 46.99) (xy 57.15 50.8)
 		)
 		(stroke
@@
 	(wire
 		(pts
-			(xy 57.15 46.99) (xy 57.15 50.8)
+			(xy 250.19 31.75) (xy 250.19 36.83)
 		)
 		(stroke
@@
 	(wire
 		(pts
-			(xy 250.19 31.75) (xy 250.19 36.83)
+			(xy 173.99 144.78) (xy 173.99 130.81)
 		)
 		(stroke
@@
 	(wire
 		(pts
-			(xy 173.99 144.78) (xy 173.99 130.81)
+			(xy 255.27 29.21) (xy 260.35 29.21)
 		)
 		(stroke
@@
 	(wire
 		(pts
-			(xy 255.27 29.21) (xy 260.35 29.21)
+			(xy 95.25 152.4) (xy 95.25 154.94)
 		)
 		(stroke
@@
 	(wire
 		(pts
-			(xy 95.25 152.4) (xy 95.25 154.94)
+			(xy 243.84 35.56) (xy 243.84 36.83)
 		)
 		(stroke
@@
 	(wire
 		(pts
-			(xy 243.84 35.56) (xy 243.84 36.83)
+			(xy 173.99 153.67) (xy 184.15 153.67)
 		)
 		(stroke
@@
 	(wire
 		(pts
+			(xy 184.15 153.67) (xy 184.15 147.32)
+		)
+		(stroke
+			(width 0)
+			(type default)
+		)
+	)
+	(wire
+		(pts
 			(xy 184.15 91.44) (xy 191.77 91.44)
 		)
@@
 	)
 	(label "PWM4"
-		(at 82.55 137.16 180)
+		(at 82.55 116.84 180)
 		(effects
 			(font
@@
 	)
 	(label "PWM3"
-		(at 82.55 134.62 180)
+		(at 82.55 121.92 180)
 		(effects
 			(font
@@
 	)
 	(label "PWM1"
-		(at 82.55 121.92 180)
+		(at 82.55 134.62 180)
 		(effects
 			(font
@@
 	)
 	(label "PWM0"
-		(at 82.55 116.84 180)
+		(at 82.55 137.16 180)
 		(effects
 			(font
@@
 			)
 		)
-		(property "Footprint" "Button_Switch_THT:SW_MEC_5GTH9"
+		(property "Footprint" "OptoDevice:Vishay_MINICAST-3Pin"
 			(at 265.43 31.75 0)
 			(effects
@@
 	(symbol
 		(lib_id "Connector_Generic:Conn_01x02")
-		(at 29.21 39.37 0)
-		(mirror y)
+		(at 29.21 41.91 180)
 		(unit 1)
 		(exclude_from_sim no)
@@
 		(on_board yes)
 		(dnp no)
-		(fields_autoplaced yes)
 		(property "Reference" "J1"
-			(at 29.21 33.02 0)
+			(at 29.21 48.26 0)
 			(effects
 				(font
@@
 		)
 		(property "Value" "XT30"
-			(at 29.21 35.56 0)
+			(at 29.21 45.72 0)
 			(effects
 				(font
@@
 		)
 		(property "Footprint" "Connector_AMASS:AMASS_XT30PW-M_1x02_P2.50mm_Horizontal"
-			(at 29.21 39.37 0)
+			(at 29.21 41.91 0)
 			(effects
 				(font
@@
 		)
 		(property "Datasheet" "~"
-			(at 29.21 39.37 0)
+			(at 29.21 41.91 0)
 			(effects
 				(font
@@
 		)
 		(property "Description" "Generic connector, single row, 01x02, script generated (kicad-library-utils/schlib/autogen/connector/)"
-			(at 29.21 39.37 0)
+			(at 29.21 41.91 0)
 			(effects
 				(font
@@
 			)
 		)
-		(property "Footprint" "Connector_PinSocket_2.54mm:PinSocket_1x03_P2.54mm_Vertical"
+		(property "Footprint" "Connector_PinHeader_2.54mm:PinHeader_1x03_P2.54mm_Vertical"
 			(at 199.39 121.666 0)
 			(effects
@@
 	)
 	(symbol
-		(lib_id "Device:C_Polarized_Small")
-		(at 240.03 72.39 0)
-		(mirror y)
-		(unit 1)
-		(exclude_from_sim no)
-		(in_bom yes)
-		(on_board yes)
-		(dnp no)
-		(property "Reference" "C4"
-			(at 237.49 70.5738 0)
-			(effects
-				(font
-					(size 1.27 1.27)
-				)
-				(justify left)
-			)
-		)
-		(property "Value" "47u"
-			(at 237.49 73.1138 0)
-			(effects
-				(font
-					(size 1.27 1.27)
-				)
-				(justify left)
-			)
-		)
-		(property "Footprint" "Capacitor_THT:CP_Radial_D5.0mm_P2.00mm"
-			(at 240.03 72.39 0)
-			(effects
-				(font
-					(size 1.27 1.27)
-				)
-				(hide yes)
-			)
-		)
-		(property "Datasheet" "~"
-			(at 240.03 72.39 0)
-			(effects
-				(font
-					(size 1.27 1.27)
-				)
-				(hide yes)
-			)
-		)
-		(property "Description" "Polarized capacitor, small symbol"
-			(at 240.03 72.39 0)
-			(effects
-				(font
-					(size 1.27 1.27)
-				)
-				(hide yes)
-			)
-		)
-		(pin "2"
-		)
-		(pin "1"
-		)
-		(instances
-			(project "main"
-				(path "/21c2240c-3034-40f0-9dbf-2fbf34e03f2d"
-					(reference "C4")
-					(unit 1)
-				)
-			)
-		)
-	)
-	(symbol
 		(lib_id "Device:LED")
 		(at 171.45 39.37 90)
@@
 	)
 	(symbol
+		(lib_id "Device:C_Polarized_Small")
+		(at 173.99 149.86 0)
+		(mirror y)
+		(unit 1)
+		(exclude_from_sim no)
+		(in_bom yes)
+		(on_board yes)
+		(dnp no)
+		(property "Reference" "C4"
+			(at 171.45 148.0438 0)
+			(effects
+				(font
+					(size 1.27 1.27)
+				)
+				(justify left)
+			)
+		)
+		(property "Value" "47u"
+			(at 171.45 150.5838 0)
+			(effects
+				(font
+					(size 1.27 1.27)
+				)
+				(justify left)
+			)
+		)
+		(property "Footprint" "Capacitor_THT:CP_Radial_D5.0mm_P2.00mm"
+			(at 173.99 149.86 0)
+			(effects
+				(font
+					(size 1.27 1.27)
+				)
+				(hide yes)
+			)
+		)
+		(property "Datasheet" "~"
+			(at 173.99 149.86 0)
+			(effects
+				(font
+					(size 1.27 1.27)
+				)
+				(hide yes)
+			)
+		)
+		(property "Description" "Polarized capacitor, small symbol"
+			(at 173.99 149.86 0)
+			(effects
+				(font
+					(size 1.27 1.27)
+				)
+				(hide yes)
+			)
+		)
+		(pin "2"
+		)
+		(pin "1"
+		)
+		(instances
+			(project "main"
+				(path "/21c2240c-3034-40f0-9dbf-2fbf34e03f2d"
+					(reference "C4")
+					(unit 1)
+				)
+			)
+		)
+	)
+	(symbol
 		(lib_id "Motor:Motor_Servo_JR")
 		(at 199.39 130.81 0)
@@
 			)
 		)
-		(property "Footprint" "Connector_PinSocket_2.54mm:PinSocket_1x03_P2.54mm_Vertical"
+		(property "Footprint" "Connector_PinHeader_2.54mm:PinHeader_1x03_P2.54mm_Vertical"
 			(at 199.39 135.636 0)
 			(effects
@@
 			)
 		)
-		(property "Footprint" "Connector_PinSocket_2.54mm:PinSocket_1x03_P2.54mm_Vertical"
+		(property "Footprint" "Connector_PinHeader_2.54mm:PinHeader_1x03_P2.54mm_Vertical"
 			(at 199.39 93.726 0)
 			(effects
@@
 			)
 		)
-		(property "Footprint" "Connector_PinSocket_2.54mm:PinSocket_1x03_P2.54mm_Vertical"
+		(property "Footprint" "Connector_PinHeader_2.54mm:PinHeader_1x03_P2.54mm_Vertical"
 			(at 199.39 149.606 0)
 			(effects
@@
 			)
 		)
-		(property "Footprint" "Connector_PinSocket_2.54mm:PinSocket_1x03_P2.54mm_Vertical"
+		(property "Footprint" "Connector_PinHeader_2.54mm:PinHeader_1x03_P2.54mm_Vertical"
 			(at 199.39 107.696 0)
 			(effects
