File: circuit/main/main.kicad_pcb (KiCad board)
At the start: 2 copper layers, 25 parts, among them J1 XT30, J2 GP1UXC41QS, J3 NeoPixel, M1 Motor_Servo_JR, M2 Motor_Servo_JR, M3 Motor_Servo_JR, M4 Motor_Servo_JR, M5 Motor_Servo_JR, SW1 SW_Push, SW3 SW_SPDT

Commit message: パターン図
Parts:
- added REF**: MountingHole_2.2mm_M2, MountingHole:MountingHole_2.2mm_M2, F.Cu at (123.0, 97.0)
- added REF**: MountingHole_2.2mm_M2, MountingHole:MountingHole_2.2mm_M2, F.Cu at (167.0, 97.0)
- added REF**: MountingHole_2.2mm_M2, MountingHole:MountingHole_2.2mm_M2, F.Cu at (123.0, 53.0)
- added REF**: MountingHole_2.2mm_M2, MountingHole:MountingHole_2.2mm_M2, F.Cu at (167.0, 53.0)
- M1, M2, M3, M4, M5: footprint Connector_PinSocket_2.54mm:PinSocket_1x03_P2.54mm_Vertical -> Connector_PinHeader_2.54mm:PinHeader_1x03_P2.54mm_Vertical
- moved D3 51.5 mm to (123.0, 87.0)
- moved R4 50.1 mm to (123.0, 82.0)
- moved U1 39.0 mm to (164.5, 70.0), turned to 90 degrees
- moved R1 38.0 mm to (133.0, 96.6), turned to -90 degrees
- moved SW1 36.9 mm to (148.2, 55.0)
- moved R3 36.4 mm to (163.6, 59.6), turned to 90 degrees
- moved C2 35.5 mm to (129.0, 95.8), turned to -90 degrees
- moved J2 35.4 mm to (135.4, 96.0)
- moved R2 33.4 mm to (167.2, 59.6), turned to 90 degrees
- moved C4 33.4 mm to (159.0, 70.0), turned to -90 degrees
- moved M5 29.6 mm to (147.9, 86.0), turned to 90 degrees
- moved A1 29.3 mm to (143.0, 89.6), turned to 180 degrees
- moved U2 28.2 mm to (159.8, 92.0), turned to 180 degrees
- moved J3 24.6 mm to (149.5, 97.0), turned to 180 degrees
- moved C1 23.8 mm to (160.0, 66.5)
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Connections:
- A1 pad 13: /PWM3 -> /PWM1
- A1 pad 14: /PWM4 -> /PWM0
- A1 pad 6: /PWM0 -> /PWM4
- A1 pad 8: /PWM1 -> /PWM3
- C4 pad 1: +BATT -> +5V
- J1 pad 1: Net-(J1-Pin_1) -> GND
- J1 pad 2: GND -> Net-(J1-Pin_2)
- R5 pad 1: Net-(J1-Pin_1) -> Net-(J1-Pin_2)
- U2 pad 4: Net-(J1-Pin_1) -> Net-(J1-Pin_2)
Routing:
- net GND: track 0.00 -> 198.3 mm, vias 0 -> 157
- net +BATT: track 0.00 -> 80.5 mm
- net /RESET: track 0.00 -> 55.9 mm
- net +5V: track 0.00 -> 44.6 mm
- net /IR_SIGNAL: track 0.00 -> 32.5 mm
- net /NEOPIXEL_SIGNAL: track 0.00 -> 31.6 mm
- net +5VD: track 0.00 -> 27.7 mm
- net Net-(J1-Pin_2): track 0.00 -> 18.3 mm
- net /PWM2: track 0.00 -> 17.2 mm
- net /PWM1: track 0.00 -> 15.1 mm
- net /PWM0: track 0.00 -> 13.0 mm
- net Net-(SW3-B): track 0.00 -> 11.9 mm, vias 0 -> 1
- net /PWM3: track 0.00 -> 11.6 mm
- net /PWM4: track 0.00 -> 11.1 mm
- net Net-(J2-Pin_3): track 0.00 -> 8.13 mm
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- added copper zone on B.Cu, net GND
- added copper zone on F.Cu, net GND
Other:
- board outline added: 50 x 50 mm

Commit message: step
Routing:
- net /IR_SIGNAL: track 32.5 -> 19.7 mm
- net GND: track 198.3 -> 186.7 mm, vias 157 -> 166
- net /NEOPIXEL_SIGNAL: track 31.6 -> 35.5 mm
- net /PWM4: track 11.1 -> 11.9 mm
- net +BATT: track 80.5 -> 81.0 mm
